Commit message: now works with odrive

File: ros2_control/bob_gazebo.ros2_control.xacro (robot description, xacro)
@@ -1,10 +1,10 @@
 <?xml version="1.0"?>
 <robot xmlns:xacro="http://www.ros.org/wiki/xacro">
-  <xacro:macro name="bob_gazebo_ros2_control" params="name prefix">
-    <ros2_control name="${name}" type="system">
+  <xacro:macro name="bob_gazebo_ros2_control" params="name">
+    <ros2_control name="bob_gazebo_ros2_control" type="system">
         <hardware>
         <plugin>gazebo_ros2_control/GazeboSystem</plugin>
         </hardware>
-            <joint name="${prefix}left_wheel_joint">
+            <joint name="left_wheel_joint">
             <command_interface name="velocity">
                 <param name="min">-1</param>
@@ -14,5 +14,5 @@
             <state_interface name="velocity"/>
             </joint>
-        <joint name="${prefix}right_wheel_joint">
+        <joint name="right_wheel_joint">
             <command_interface name="velocity">
                 <param name="min">-1</param>

File: urdf/bob.urdf.xacro (robot description, xacro)
@@ -2,5 +2,4 @@
 <!-- Basic differential drive mobile base -->
 <robot xmlns:xacro="http://www.ros.org/wiki/xacro" name="bob">
-  <xacro:arg name="prefix" default="" />
   <xacro:arg name="simulated" default="true" />
   <!-- Import Rviz colors -->
@@ -8,10 +7,10 @@
   <xacro:include filename="$(find bob_description)/urdf/bob_description.urdf.xacro" />
   <!-- Call macro to summon bob -->
-  <xacro:summon_bob prefix="$(arg prefix)" />
+  <xacro:summon_bob/>
   <!-- If simulating in gazebo, load simulated hardware interfaces and joint state broadcasters -->
   <xacro:if value="$(arg simulated)">
     <xacro:include filename="$(find bob_description)/ros2_control/bob_gazebo.ros2_control.xacro" />
     <xacro:bob_gazebo_ros2_control
-      name="bob" prefix="$(arg prefix)" />
+      name="bob_gazebo_control" />
     <gazebo>
       <plugin filename="libgazebo_ros2_control.so" name="gazebo_ros2_control">
@@ -20,9 +19,9 @@
     </gazebo>
   </xacro:if>
-  <!-- Else use the actual hardware interfaces (currently defaulted to a dummy one) -->
+  <!-- Else use the actual hardware interfaces -->
   <xacro:unless value="$(arg simulated)">
-    <xacro:include filename="$(find bob_description)/ros2_control/bob.ros2_control.xacro" />
+    <xacro:include filename="$(find bob_description)/ros2_control/bob_odrive_ros2_control.xacro" />
     <xacro:bob_ros2_control
-      name="bob" prefix="$(arg prefix)" />
+      name="bob_control" />
   </xacro:unless>
 </robot>

File: urdf/bob_description.urdf.xacro (robot description, xacro)
@@ -1,5 +1,5 @@
 <?xml version="1.0"?>
 <robot xmlns:xacro="http://www.ros.org/wiki/xacro">
-  <xacro:macro name="summon_bob" params="prefix">
+  <xacro:macro name="summon_bob">
     <!-- Constants for robot dimensions -->
     <xacro:property name="PI" value="3.1415926535897931"/>
@@ -16,5 +16,5 @@
     <xacro:property name="x_offset" value="0.2" />
     <!-- Base Link -->
-    <link name="${prefix}base_link">
+    <link name="base_link">
       <collision>
         <origin xyz="0 0 ${base_height/2}" rpy="0 0 0"/>
@@ -39,7 +39,7 @@
         </inertial>
     </link>
-    <joint name="${prefix}left_wheel_joint" type="continuous">
-      <parent link="${prefix}base_link"/>
-      <child link="${prefix}left_wheel"/>
+    <joint name="left_wheel_joint" type="continuous">
+      <parent link="base_link"/>
+      <child link="left_wheel"/>
       <origin xyz="-${x_offset} -${base_width/2} ${z_offset}" rpy="-${PI/2} 0 0"/>
       <axis xyz="0 0 1"/>
@@ -47,5 +47,5 @@
     </joint>
     <!-- left wheel Link -->
-    <link name="${prefix}left_wheel">
+    <link name="left_wheel">
       <collision>
         <origin xyz="0 0 0" rpy="0 0 0"/>
@@ -70,7 +70,7 @@
       </inertial>
     </link>
-    <joint name="${prefix}right_wheel_joint" type="continuous">
-      <parent link="${prefix}base_link"/>
-      <child link="${prefix}right_wheel"/>
+    <joint name="right_wheel_joint" type="continuous">
+      <parent link="base_link"/>
+      <child link="right_wheel"/>
       <origin xyz="-${x_offset} ${base_width/2} ${z_offset}" rpy="-${PI/2} 0 0"/>
       <axis xyz="0 0 1"/>
@@ -78,5 +78,5 @@
     </joint>
       <!-- right wheel Link -->
-    <link name="${prefix}right_wheel">
+    <link name="right_wheel">
       <collision>
         <origin xyz="0 0 0" rpy="0 0 0"/>
@@ -101,7 +101,7 @@
       </inertial>
     </link>
-    <joint name="${prefix}front_left_wheel_joint" type="fixed">
-      <parent link="${prefix}base_link"/>
-      <child link="${prefix}front_left_wheel"/>
+    <joint name="front_left_wheel_joint" type="fixed">
+      <parent link="base_link"/>
+      <child link="front_left_wheel"/>
       <origin xyz="${x_offset} -${base_width/2} ${z_offset}" rpy="-${PI/2} 0 0"/>
     </joint>
@@ -132,7 +132,7 @@
       <mu2 value="0.0"/>
     </gazebo>
-    <joint name="${prefix}front_right_wheel_joint" type="fixed">
-      <parent link="${prefix}base_link"/>
-      <child link="${prefix}front_right_wheel"/>
+    <joint name="front_right_wheel_joint" type="fixed">
+      <parent link="base_link"/>
+      <child link="front_right_wheel"/>
       <origin xyz="${x_offset} ${base_width/2} ${z_offset}" rpy="-${PI/2} 0 0"/>
     </joint>

Commit message: added transmission

File: ros2_control/bob_gazebo.ros2_control.xacro (robot description, xacro)
@@ -22,4 +22,16 @@
             <state_interface name="velocity"/>
         </joint>
+        <transmission name="left_wheel_transmission">
+            <plugin>transmission_interface/SimpleTransmission</plugin>
+            <joint name="left_wheel_joint" role="left_wheel_joint">
+                <mechanical_reduction>5</mechanical_reduction>
+            </joint>
+        </transmission>
+        <transmission name="right_wheel_transmission">
+            <plugin>transmission_interface/SimpleTransmission</plugin>
+            <joint name="right_wheel_joint" role="right_wheel_joint">
+                <mechanical_reduction>5</mechanical_reduction>
+            </joint>
+        </transmission>
     </ros2_control>
   </xacro:macro>
