Commit message: now doesnt jank up the sim

File: urdf/bob.urdf.xacro (robot description, xacro)
@@ -4,4 +4,6 @@
   <xacro:arg name="prefix" default="" />
   <xacro:arg name="simulated" default="true" />
+  <!-- Import Rviz colors -->
+  <xacro:include filename="$(find bob_description)/gazebo/bob_materials.xacro" />
   <xacro:include filename="$(find bob_description)/urdf/bob_description.urdf.xacro" />
   <!-- Call macro to summon bob -->

File: urdf/bob_description.urdf.xacro (robot description, xacro)
@@ -4,20 +4,21 @@
     <!-- Constants for robot dimensions -->
     <xacro:property name="PI" value="3.1415926535897931"/>
-    <xacro:property name="base_mass" value="0.3" /> <!-- arbitrary value for base mass -->
-    <xacro:property name="base_width" value="0.1" />
-    <xacro:property name="base_length" value="0.1" />
-    <xacro:property name="base_height" value="0.05" />
-    <xacro:property name="wheel_mass" value="0.3" /> <!-- arbitrary value for wheel mass -->
-    <xacro:property name="wheel_len" value="0.020" />
-    <xacro:property name="wheel_radius" value="0.015" />
+    <xacro:property name="base_mass" value="30" /> <!-- arbitrary value for base mass -->
+    <xacro:property name="base_width" value="0.45" />
+    <xacro:property name="base_length" value="0.6" />
+    <xacro:property name="base_height" value="0.5" />
+    <xacro:property name="wheel_mass" value="0.5" /> <!-- arbitrary value for wheel mass -->
+    <xacro:property name="wheel_len" value="0.05" />
+    <xacro:property name="wheel_radius" value="0.1" />
     <xacro:property name="caster_wheel_mass" value="0.1" /> <!-- arbitrary value for caster wheel mass -->
     <xacro:property name="caster_wheel_radius" value="0.015" />
-    <xacro:property name="z_offset" value="-${base_height/2}" /> <!-- Space btw top of beam and the each joint -->
+    <xacro:property name="z_offset" value="0.05" /> <!-- Space btw top of beam and the each joint -->
+    <xacro:property name="x_offset" value="0.2" />
     <!-- Base Link -->
     <link name="${prefix}base_link">
       <collision>
-        <origin xyz="0 0 0" rpy="0 0 0"/>
+        <origin xyz="0 0 ${base_height/2}" rpy="0 0 0"/>
         <geometry>
-          <box size="${base_width} ${base_length} ${base_height}"/>
+          <box size="${base_length} ${base_width} ${base_height}"/>
         </geometry>
       </collision>
@@ -25,10 +26,10 @@
         <origin xyz="0 0 ${base_height/2}" rpy="0 0 0"/>
         <geometry>
-          <box size="${base_width} ${base_length} ${base_height}"/>
+          <box size="${base_length} ${base_width} ${base_height}"/>
         </geometry>
-        <material name="orange"/>
+        <material name="grey"/>
       </visual>
       <inertial>
-        <origin xyz="0 0 0" rpy="0 0 0"/>
+        <origin xyz="0 0 ${base_height/2}" rpy="0 0 0"/>
         <mass value="${base_mass}"/>
         <inertia
@@ -41,6 +42,6 @@
       <parent link="${prefix}base_link"/>
       <child link="${prefix}left_wheel"/>
-      <origin xyz="0 -${base_width/2} ${z_offset}" rpy="0 0 0"/>
-      <axis xyz="0 1 0"/>
+      <origin xyz="-${x_offset} -${base_width/2} ${z_offset}" rpy="-${PI/2} 0 0"/>
+      <axis xyz="0 0 1"/>
       <dynamics damping="0.2"/>
     </joint>
@@ -48,5 +49,5 @@
     <link name="${prefix}left_wheel">
       <collision>
-        <origin xyz="0 0 0" rpy="${PI/2} 0 0"/>
+        <origin xyz="0 0 0" rpy="0 0 0"/>
         <geometry>
           <cylinder length="${wheel_len}" radius="${wheel_radius}"/>
@@ -54,5 +55,5 @@
       </collision>
       <visual>
-        <origin xyz="0 0 0" rpy="${PI/2} 0 0"/>
+        <origin xyz="0 0 0" rpy="0 0 0"/>
         <geometry>
           <cylinder length="${wheel_len}" radius="${wheel_radius}"/>
@@ -61,5 +62,5 @@
       </visual>
       <inertial>
-        <origin xyz="0 0 0" rpy="${PI/2} 0 0"/>
+        <origin xyz="0 0 0" rpy="0 0 0"/>
         <mass value="${wheel_mass}"/>
         <inertia
@@ -72,6 +73,6 @@
       <parent link="${prefix}base_link"/>
       <child link="${prefix}right_wheel"/>
-      <origin xyz="0 ${base_width/2} ${z_offset}" rpy="0 0 0"/>
-      <axis xyz="0 1 0"/>
+      <origin xyz="-${x_offset} ${base_width/2} ${z_offset}" rpy="-${PI/2} 0 0"/>
+      <axis xyz="0 0 1"/>
       <dynamics damping="0.2"/>
     </joint>
@@ -79,5 +80,5 @@
     <link name="${prefix}right_wheel">
       <collision>
-        <origin xyz="0 0 0" rpy="${PI/2} 0 0"/>
+        <origin xyz="0 0 0" rpy="0 0 0"/>
         <geometry>
           <cylinder length="${wheel_len}" radius="${wheel_radius}"/>
@@ -85,5 +86,5 @@
       </collision>
       <visual>
-        <origin xyz="0 0 0" rpy="${PI/2} 0 0"/>
+        <origin xyz="0 0 0" rpy="0 0 0"/>
         <geometry>
           <cylinder length="${wheel_len}" radius="${wheel_radius}"/>
@@ -92,5 +93,5 @@
       </visual>
       <inertial>
-        <origin xyz="0 0 0" rpy="${PI/2} 0 0"/>
+        <origin xyz="0 0 0" rpy="0 0 0"/>
         <mass value="${wheel_mass}"/>
         <inertia
@@ -100,21 +101,19 @@
       </inertial>
     </link>
-    <joint name="${prefix}caster_frontal_wheel_joint" type="fixed">
+    <joint name="${prefix}front_left_wheel_joint" type="fixed">
       <parent link="${prefix}base_link"/>
-      <child link="${prefix}caster_frontal_wheel"/>
-      <origin xyz="${base_width/2 - caster_wheel_radius} 0 ${z_offset}" rpy="0 0 0"/>
+      <child link="${prefix}front_left_wheel"/>
+      <origin xyz="${x_offset} -${base_width/2} ${z_offset}" rpy="-${PI/2} 0 0"/>
     </joint>
-    <!-- caster frontal wheel Link -->
-    <link name="${prefix}caster_frontal_wheel">
+    <!-- front left wheel Link -->
+    <link name="front_left_wheel">
       <collision>
-        <origin xyz="0 0 0" rpy="0 0 0"/>
         <geometry>
-          <sphere radius="${caster_wheel_radius}"/>
+          <cylinder length="${wheel_len}" radius="${wheel_radius}"/>
         </geometry>
       </collision>
       <visual>
-        <origin xyz="0 0 0" rpy="0 0 0"/>
         <geometry>
-          <sphere radius="${caster_wheel_radius}"/>
+          <cylinder length="${wheel_len}" radius="${wheel_radius}"/>
         </geometry>
         <material name="white"/>
@@ -122,28 +121,30 @@
       <inertial>
         <origin xyz="0 0 0" rpy="0 0 0"/>
-        <mass value="${caster_wheel_mass}"/>
+        <mass value="${wheel_mass}"/>
         <inertia
-          ixx="${caster_wheel_mass * 0.4 * (caster_wheel_radius * caster_wheel_radius)}" ixy="0.0" ixz="0.0"
-          iyy="${caster_wheel_mass * 0.4 * (caster_wheel_radius * caster_wheel_radius)}" iyz="0.0"
-          izz="${caster_wheel_mass * 0.4 * (caster_wheel_radius * caster_wheel_radius)}"/>
+          ixx="${wheel_mass / 12.0 * (3*wheel_radius + wheel_len*wheel_len)}" ixy="0.0" ixz="0.0"
+          iyy="${wheel_mass / 12.0 * wheel_radius*wheel_radius}" iyz="0.0"
+          izz="${wheel_mass / 12.0 * wheel_radius*wheel_radius}"/>
       </inertial>
     </link>
-    <joint name="${prefix}caster_rear_wheel_joint" type="fixed">
+    <gazebo reference="front_left_wheel">
+      <mu1 value="0.0"/>
+      <mu2 value="0.0"/>
+    </gazebo>
+    <joint name="${prefix}front_right_wheel_joint" type="fixed">
       <parent link="${prefix}base_link"/>
-      <child link="${prefix}caster_rear_wheel"/>
-      <origin xyz="${-base_width/2 + caster_wheel_radius} 0 ${z_offset}" rpy="0 0 0"/>
+      <child link="${prefix}front_right_wheel"/>
+      <origin xyz="${x_offset} ${base_width/2} ${z_offset}" rpy="-${PI/2} 0 0"/>
     </joint>
-    <!-- caster rear wheel Link -->
-    <link name="${prefix}caster_rear_wheel">
+    <!-- front right wheel Link -->
+    <link name="front_right_wheel">
       <collision>
-        <origin xyz="0 0 0" rpy="0 0 0"/>
         <geometry>
-          <sphere radius="${caster_wheel_radius}"/>
+          <cylinder length="${wheel_len}" radius="${wheel_radius}"/>
         </geometry>
       </collision>
       <visual>
-        <origin xyz="0 0 0" rpy="0 0 0"/>
         <geometry>
-          <sphere radius="${caster_wheel_radius}"/>
+          <cylinder length="${wheel_len}" radius="${wheel_radius}"/>
         </geometry>
         <material name="white"/>
@@ -151,11 +152,15 @@
       <inertial>
         <origin xyz="0 0 0" rpy="0 0 0"/>
-        <mass value="${caster_wheel_mass}"/>
+        <mass value="${wheel_mass}"/>
         <inertia
-          ixx="${caster_wheel_mass * 0.4 * (caster_wheel_radius * caster_wheel_radius)}" ixy="0.0" ixz="0.0"
-          iyy="${caster_wheel_mass * 0.4 * (caster_wheel_radius * caster_wheel_radius)}" iyz="0.0"
-          izz="${caster_wheel_mass * 0.4 * (caster_wheel_radius * caster_wheel_radius)}"/>
+          ixx="${wheel_mass / 12.0 * (3*wheel_radius + wheel_len*wheel_len)}" ixy="0.0" ixz="0.0"
+          iyy="${wheel_mass / 12.0 * wheel_radius*wheel_radius}" iyz="0.0"
+          izz="${wheel_mass / 12.0 * wheel_radius*wheel_radius}"/>
       </inertial>
     </link>
+    <gazebo reference="front_right_wheel">
+      <mu1 value="0.0"/>
+      <mu2 value="0.0"/>
+    </gazebo>
   </xacro:macro>
 </robot>

Commit message: sim imu

File: urdf/bob.urdf.xacro (robot description, xacro)
@@ -8,9 +8,10 @@
   <!-- Call macro to summon bob -->
   <xacro:summon_bob/>
-  <!-- If simulating in gazebo, load simulated hardware interfaces and joint state broadcasters -->
+  <!-- If simulating in gazebo, load simulated hardware interfaces, senso and joint state broadcasters -->
   <xacro:if value="$(arg simulated)">
     <xacro:include filename="$(find bob_description)/ros2_control/bob_gazebo_ros2_control.xacro" />
-    <xacro:bob_gazebo_ros2_control
-      name="bob_gazebo_control" />
+    <xacro:include filename="$(find bob_description)/gazebo/bob_gazebo_sensors.xacro" />
+    <xacro:bob_gazebo_ros2_control name="bob_gazebo_control" />
+    <xacro:bob_gazebo_sensors />
     <gazebo>
       <plugin filename="libgazebo_ros2_control.so" name="gazebo_ros2_control">

File: urdf/bob_description.urdf.xacro (robot description, xacro)
@@ -163,4 +163,11 @@
       <mu2 value="0.0"/>
     </gazebo>
+    <!-- IMU-->
+    <link name="imu_link"/>
+    <joint name="imu_joint" type="fixed">
+      <parent link="base_link"/>
+      <child link="imu_link"/>
+      <origin xyz="0 0 0"/>
+    </joint>
   </xacro:macro>
 </robot>

Commit message: bob town simulation

File: urdf/bob.urdf.xacro (robot description, xacro)
@@ -3,7 +3,8 @@
 <robot xmlns:xacro="http://www.ros.org/wiki/xacro" name="bob">
   <xacro:arg name="simulated" default="true" />
-  <!-- Import Rviz colors -->
+  <!-- Import xacro files -->
   <xacro:include filename="$(find bob_description)/gazebo/bob_materials.xacro" />
   <xacro:include filename="$(find bob_description)/urdf/bob_description.urdf.xacro" />
+  <xacro:include filename="$(find bob_description)/sensors/intel_d435.xacro" />
   <!-- Call macro to summon bob -->
   <xacro:summon_bob/>
@@ -11,7 +12,7 @@
   <xacro:if value="$(arg simulated)">
     <xacro:include filename="$(find bob_description)/ros2_control/bob_gazebo_ros2_control.xacro" />
-    <xacro:include filename="$(find bob_description)/gazebo/bob_gazebo_sensors.xacro" />
+    <xacro:include filename="$(find bob_description)/gazebo/bob_gazebo_imu.xacro" />
     <xacro:bob_gazebo_ros2_control name="bob_gazebo_control" />
-    <xacro:bob_gazebo_sensors />
+    <xacro:bob_gazebo_imu />
     <gazebo>
       <plugin filename="libgazebo_ros2_control.so" name="gazebo_ros2_control">
@@ -26,3 +27,8 @@
       name="bob_control" />
   </xacro:unless>
+  <!-- Slap in the intel d435-->
+  <!-- <xacro:intel_d435 parent="base_link">
+     <origin xyz="0.35 0 0.3" />
+  </xacro:intel_d435> -->
+  <!--  NOTE set to pose param from model.sdf -->
 </robot>
